File: Hardware/Kicad_SPIP/Kicad_SPIP.kicad_pcb (KiCad board)
At the start: 4 copper layers, 40 x 60 mm, 60 parts, among them J1 Conn_01x02, J2 Conn_ST_STDC14, J3 Conn_01x03, J4 Conn_01x04, J5 Conn_01x06, J6 Conn_01x06, J7 Conn_01x06, SW1 SW_Push, SW2 SW_Push, SW3 SW_Push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

Commit message: pcb rootage
Parts:
- removed H5, H6, H7, H8: MountingHole_Pad, MountingHole:MountingHole_3.2mm_M3_Pad_Via
- C17: footprint LED_SMD:LED_0603_1608Metric -> Capacitor_SMD:C_0402_1005Metric
- J4: footprint Connector_JST:JST_PH_B3B-PH-K_1x03_P2.00mm_Vertical -> Connector_JST:JST_PH_B4B-PH-K_1x04_P2.00mm_Vertical
- J5: footprint Connector_JST:JST_PH_B3B-PH-K_1x03_P2.00mm_Vertical -> Connector_JST:JST_PH_B6B-PH-K_1x06_P2.00mm_Vertical
- moved SW1 213.5 mm to (46.7, 77.9), turned to 90 degrees
- moved R8 112.3 mm to (81.0, 62.4), turned to -90 degrees
- moved R9 110.5 mm to (82.8, 64.3)
- moved C9 109.3 mm to (81.0, 60.0), turned to -90 degrees
- moved J4 103.4 mm to (49.9, 56.4), turned to -90 degrees
- moved SW2 103.0 mm to (83.3, 61.2), turned to -90 degrees
- moved C10 100.5 mm to (53.0, 57.2), turned to -90 degrees
- moved C8 93.2 mm to (58.2, 90.9)
- moved J3 85.8 mm to (57.0, 94.0)
- moved C13 84.6 mm to (81.0, 66.2), turned to -90 degrees
- moved R12 81.7 mm to (81.0, 68.6), turned to -90 degrees
- moved SW3 78.5 mm to (83.3, 67.4), turned to -90 degrees
- moved R14 78.1 mm to (82.8, 70.5)
- moved J5 67.4 mm to (70.0, 49.0), turned to 180 degrees
- moved C14 67.4 mm to (69.2, 52.0), turned to 180 degrees
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Routing:
- net /RIGHT_ENC_B: track 0.00 -> 42.4 mm, vias 0 -> 2
- net /RIGHT_ENC_A: track 0.00 -> 42.0 mm, vias 0 -> 2
- net /LEFT_ENC_A: track 0.00 -> 40.1 mm, vias 0 -> 1
- net /LEFT_ENC_B: track 0.00 -> 40.0 mm, vias 0 -> 1
- net /AIN1: track 0.00 -> 37.7 mm, vias 0 -> 2
- net /AIN2: track 0.00 -> 35.8 mm, vias 0 -> 2
- net /X4: track 0.00 -> 32.6 mm, vias 0 -> 1
- net +3.3V: track 15.2 -> 47.2 mm, vias 7 -> 22
- net /X3: track 0.00 -> 30.5 mm, vias 0 -> 1
- net /X2: track 0.00 -> 30.1 mm, vias 0 -> 1
- net /X1: track 0.00 -> 27.8 mm, vias 0 -> 1
- net /TRIGG: track 0.00 -> 27.6 mm, vias 0 -> 2
- net /ECHO: track 0.00 -> 27.2 mm, vias 0 -> 2
- net /JTMS/SWDIO: track 0.00 -> 26.5 mm
- net /DATA: track 0.00 -> 26.4 mm, vias 0 -> 2
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
Commit message: derniere version du PCB Layout
Routing:
- net GND: vias 62 -> 185
Other:
- board text added: "ANDRIEU"
- board text added: "MAHI"
- board text added: "Projet SPIP :"
- board text added: "WANTIEZ"

Commit message: pin ultrason Kicad déplacé & code encoder & moteur v2
Parts:
- moved J4 5.35 mm to (55.2, 57.1), turned to 180 degrees
- moved C10 3.36 mm to (54.4, 60.2), turned to 180 degrees
Routing:
- net /ECHO: track 27.2 -> 28.6 mm
- net GND: vias 185 -> 194
- net (no net): vias 0 -> 1
